File: wanhao extruder pcb.sch (KiCad schematic (older format))
At the start: 8 parts, among them J1 Conn_02x10_Counter_Clockwise, T0 Conn_01x02

Commit message: Updates to extruder board
Parts:
- added HE0-0: Conn_01x02, Connector_JST:JST_XH_B2B-XH-A_1x02_P2.50mm_Vertical, symbol Connector_Generic:Conn_01x02
- renumbered HE0 to HE0-1
Connections:
- net 24V: now also HE0-0.1 (Pin_1)
- net HEATGND: now also HE0-0.2 (Pin_2)
