File: skr13-interface-wiring.sch (KiCad schematic (older format))
At the start: 22 parts

Commit message: Updates & missing elements in skr1.3 interface wiring
Parts:
- added SKR-E0MOT, SKR-XMOT, SKR-YMOT, SKR-ZMOT?, XMOT: Conn_01x04, Connector_JST:JST_XH_B4B-XH-A_1x04_P2.50mm_Vertical, symbol Connector_Generic:Conn_01x04
- added SKR-HBED: Conn_01x02, Connector_JST:JST_XH_B2B-XH-A_1x02_P2.50mm_Vertical, symbol Connector_Generic:Conn_01x02
- added SKR-TH?: SKR-HE0, Connector_JST:JST_XH_B2B-XH-A_1x02_P2.50mm_Vertical, symbol Connector_Generic:Conn_01x02
- gave numbers to parts that had none: 1
Connections:
- net 24V: now also SKR-HBED.1 (Pin_1)
- net HBED24V: now also SKR-TH?.1 (Pin_1)
- net HBEDGND: now also SKR-TH?.2 (Pin_2)
- net HEATGND: now also SKR-HBED.2 (Pin_2)
- net Y-1A: now also SKR-YMOT.3 (Pin_3)
- net Y-1B: now also SKR-YMOT.4 (Pin_4)
- net Y-2A: now also SKR-YMOT.2 (Pin_2)
- net Y-2B: now also SKR-YMOT.1 (Pin_1)
- net 1A renamed E0-1A
- net E0-1A: now also SKR-E0MOT.3 (Pin_3)
- net 1B renamed E0-1B
- net E0-1B: now also SKR-E0MOT.4 (Pin_4)
- net 2A renamed E0-2A
- net E0-2A: now also SKR-E0MOT.2 (Pin_2)
- net 2B renamed E0-2B
- net E0-2B: now also SKR-E0MOT.1 (Pin_1)
- new net X-1A: SKR-XMOT.3 (Pin_3), XMOT.3 (Pin_3)
- new net X-1B: SKR-XMOT.4 (Pin_4), XMOT.4 (Pin_4)
- new net X-2A: SKR-XMOT.2 (Pin_2), XMOT.2 (Pin_2)
- new net X-2B: SKR-XMOT.1 (Pin_1), XMOT.1 (Pin_1)
- new net Z-1A: SKR-ZMOT?.3 (Pin_3)
- new net Z-1B: SKR-ZMOT?.4 (Pin_4)
- new net Z-2A: SKR-ZMOT?.2 (Pin_2)
- new net Z-2B: SKR-ZMOT?.1 (Pin_1)
Other:
- moved on the sheet: AUX?, HBED?, TBED?, Y-?, Z-?
